Commit message: 官方新规则落地(第 1 批): 立牌 5x15x5mm/16 个 · 雷达降高+前装 · 灯箱 5cm/黄 5s · 地图修正
一、按官方规则改的场景/参数
 1) 立牌: 高 15 cm x 宽 5 cm x 厚 5 mm (官方统一尺寸, 原为按各图轮廓比 39~70mm/3mm),
    人物按 contain 居中放进 5:15 板面, 碰撞体与雷达反射面都是 5x15。
 2) 立牌数量: 10 -> **16 = 14 社区 + 2 非社区** (官方要求 >=14+2),
    A 街区 10 (北5+南4+西1, 含 F1) / B 街区 6 (北4+东2, 含 F2) —— 两个街区都有两类人,
    也不存在"一个街区只有 1 个人偶"。模型不用新建(官方素材正好 16+2)。
 3) 雷达高度: 0.20 -> **车体前方 0.32 m 支架上的 0.12 m**, 扫描 ±140°。
    为什么这么绕: 官方要求"立牌能被雷达扫到", 但实测出硬约束 ——
      车体箱体 z 范围 0.0276~0.1673 (height 0.1397 + center_offset.z 0.0974),
      立牌顶面只有 0.150 -> "在车体上方"与"扫到立牌"不可能同时满足;
      而降到 0.12 又会让雷达**埋在车体内部**, 每个方向先打自己的壳:
      实测 AMCL 自信漂移 2.6 m、激光对墙反推偏 0.43 m、巡航 0/17。
    最终: 前装 0.32 m(车体遮挡只剩 ±40°) + 扫 ±140°(避开自遮挡且给 AMCL 留足墙面)。
 4) 红绿灯: 箱体厚度 8 -> 5 cm (官方); 三色时长 黄 3 -> **5 s** (官方 红10/黄5/绿15),
    验收的循环观察窗口 22 -> 35 s。
 5) 项目里一直缺的官方素材根因: 脚本读 ~/复赛资料, 而素材在 D:\BaiduNetdiskDownload\复赛资料 ->
    做软链修好 (gen_standees / setup_cars 都靠它)。

二、修掉两个真 bug (都是这次改动暴露的)
 1) **gen_map_from_arena.py 有 y 镜像 bug**: PGM 行序与 map_server 约定相反, 地图整体沿 y 翻转。
    以前地图里只有四面**对称**的墙所以从没暴露; 这次加入 A/B 街区等**非对称**障碍后,
    障碍落到了镜像位置(实测 A 街区被标成可通行、起点被标成障碍)。已加 [::-1] 修正。
 2) **地图原来把墙以内全当自由空间** -> 规划器没有理由不进街区; 雷达看得见立牌后,
    街区边上的立牌把车道"挤窄", 规划器就从街区内部绕 -> AMCL 在街区里漂 2.6 m。
    新增 config/map_obstacles.yaml (A/B 街区 + 右侧停车列 = 不可通行) 并重新生成地图,
    训练"不得压越车道线"这件事由地图结构性保证。

三、验收现状: 通过 8 项 / 失败 2 项
 通过: 场景(16 立牌) · 红绿灯 6/6 · 定位 1.36cm · 雷达位姿 13.1mm ·
       倒车入库 0.0155m/0.96° · **车道合规 23954 帧 0 帧压线** · 通行闸两项
 失败: 巡航 11/17 (街区障碍标成不可通行后, 贴边的航点落进膨胀代价区, 规划器放弃);
       识别三项 (巡航没跑全 + 视觉模型还是按旧立牌/旧灯箱训练的, 必须重训)

四、下一步(未做)
 官方材质(用官方 6 张红绿灯照片做灯罩) · 随机车牌(自己生成, 不用官方那三张图) ·
 国赛元素(楼宇/电动车/垃圾桶/指示牌) · 机器人外观重设计(保留尺寸与运动学) ·
 重训三个模型 · 贴边航点调参使之可达。

File: src/competition_robot/urdf/competition_robot.urdf (robot description, URDF)
Before this commit: robot competition_robot, 9 links, 8 joints
Joints:
- joint laser_joint: origin xyz=0.13374 0 0.2 rpy=0 0 0 -> xyz=0.32 0 0.12 rpy=0 0 0

Commit message: 机器人最终形态: 自研低顶架外观 + 雷达装顶板上方(恢复整圈) · 相机位不变
一、为什么要改
 1) 官方规则: "机器人自己建模可以加分, 用开源/现成机器人扣分"。而仿真机器人的外观
    一直用的是**实车导出的 STL** (mecanum/base_link.STL, 连车上的 OLED 都看得见) ——
    等于直接搬了比赛公司的车, 拿不到自建分。
 2) 官方规则: 立牌(15 cm)必须"能被雷达扫到"。实测算出硬约束:
      实车壳体 z 范围 0.0276~0.1673 (height 0.1397 + center_offset.z 0.0974)
      立牌顶面 0.150
    -> "雷达装在车体上方"(>0.1673) 与 "扫描平面穿过立牌"(<0.150) 不可能同时满足;
       降到 0.12 又会让雷达埋进壳里 (整圈扫先打自己: AMCL 自信漂移 2.6 m、
       激光对墙偏 0.43 m、巡航 0/17)。

二、最终形态 (一个改动同时解决两件事)
 * simulation.visual_style: mesh -> **primitives**，车壳改为**自研低顶架**:
     底板 0.330x0.215x0.008 @z0.068 + 四立柱 14mm + 顶板 0.310x0.190x0.006 @z0.112
     + 电池盒 + 工控机盒 + 队伍标牌(橙色) + 相机立柱   顶面 = 0.115 m
 * chassis.height 0.1397 -> **0.118**，center_offset.z 0.0974 -> 0.0590
   (运动学与 footprint 不变: 轮径 48.5 / 轮距 290.8 / 前轴 +127.2 / 后轴 -79.8 全部保留)
 * sensors.lidar2d.mount -> **[0.020, 0.0, 0.140]**，use_full_circle: **true**
   顶面 0.115 < 0.140 < 立牌顶面 0.150 -> 既不被自身遮挡(可整圈 360°) 又能扫到立牌
 * **相机安装位保持不变** (0.14914, -0.0005, 0.19998) -> 10 个识别点位与 17 站路线不用重算

三、验收结果 (新形态)
 通过: 场景(16 立牌) · 红绿灯 6/6 · 定位 1.35cm · **雷达位姿 1.1mm** ·
       倒车入库 0.0127m/0.69° · **车道合规 0/25595 帧** · 通行闸(强制红灯)
 仍在修: 巡航 15/17 (两站落在街区障碍的膨胀代价区, 待导航调参) ·
       立牌识别 (视觉模型按旧 5x15 之前的立牌训练, 待重训) · 巡航放行 1/2 (上一条的连带)

新增 docs/robot_form.png (外观图, 由 tools/draw_robot.py 从 URDF 盒体直接画)

File: src/competition_robot/urdf/competition_robot.urdf (robot description, URDF)
Before this commit: robot competition_robot, 9 links, 8 joints
Links:
- link base_link: geometry collision box size=0.3334 0.2187 0.118; visual box size=0.002 0.100 0.028
- link camera_link: geometry collision box size=0.03 0.10 0.03; visual box size=0.03 0.10 0.03
- link fl_wheel_link: geometry collision cylinder length=0.0506 radius=0.0485; visual cylinder length=0.0506 radius=0.03492
- link fr_wheel_link: geometry collision cylinder length=0.0506 radius=0.0485; visual cylinder length=0.0506 radius=0.03492
- link imu_link: geometry collision box size=0.04 0.04 0.015; visual box size=0.04 0.04 0.015
- link laser_link: geometry collision cylinder length=0.05 radius=0.05; visual cylinder length=0.05 radius=0.05
- link rl_wheel_link: geometry collision cylinder length=0.0506 radius=0.0485; visual cylinder length=0.0506 radius=0.03492
- link rr_wheel_link: geometry collision cylinder length=0.0506 radius=0.0485; visual cylinder length=0.0506 radius=0.03492
Joints:
- joint laser_joint: origin xyz=0.32 0 0.12 rpy=0 0 0 -> xyz=0.02 0 0.14 rpy=0 0 0

Commit message: 相机支架改后方立柱+悬臂: 原来挡雷达正前方, 是巡航 2 站失败的根因 (17/17 恢复)
问题 (用户发现): 原先的相机立柱 cam_post 是 20x20mm、z 0.115~0.200, 而雷达扫描平面
在 z=0.14 —— 立柱**穿过扫描平面且正在雷达正前方 12.9 cm**:
  * 挡住正前方约 ±4.8° (约 9°), 这些光束返回 ~0.13 m
  * 该回波落在车体自己的 footprint 内 (车头到 0.193), 于是局部代价地图把
    "正前方 13 cm" 标成障碍 -> 贴边航点更容易被 DWA 判为不可行

修法: 立柱挪到**雷达后方** 0.145 m 处 (只挡后方 ±2°, 车尾方向对前进与 AMCL 无影响),
再用悬臂 (z=0.2265, 在扫描平面上方) 把相机往前吊到原安装位。
复核结果: 除雷达自身外, 没有任何部件穿过 z=0.14 扫描平面。
相机安装位不变 (0.14914, -0.000497, 0.19998) -> 识别点位/路线不用重算。

验收 (同一形态, 只改支架): **通过 9 项 / 失败 1 项**
  **巡航 17/17** (原 15/17) · 雷达位姿 0.6mm · 定位 1.34cm · 车道合规 0/20935 帧 ·
  倒车入库 0.0131m/0.56° · 通行闸 放行2次误拦0 + 强制红灯停到超时 · 红绿灯 6/6 ·
  车牌 3/3 · 双通道 5/5
只剩立牌识别 (1/5): 视觉模型还是按旧立牌训练的, 待重训 (已规划)。

File: src/competition_robot/urdf/competition_robot.urdf (robot description, URDF)
Before this commit: robot competition_robot, 9 links, 8 joints
Links:
- link base_link: geometry collision box size=0.3334 0.2187 0.118; visual box size=0.002 0.100 0.028
